File: KiCAD/Backglass.sch (KiCad schematic (older format))
At the start: 54 parts, among them J1 IO Header, J11 Header_ICSP_AVR, J12 Header_ICSP_AVR, J13 Header_ICSP_AVR, J2 RAMP Header, J3 LOSE Header, J4 Micro_USB_Connector, J5 Batteries, Q1 MOSFET_N_E, Q2 MOSFET_N_E+P_E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

Commit message: Fixed audio output, reduced power consumption
Removed half-bridge and associated components, modified resistor values
to drive LEDs dimmer (and now within power specs for the 48PB).
Parts:
- removed C4: 220u, M_Through-hole:C_6.3-2.5mm, symbol CP
- removed Q1: MOSFET_N_E, M_SMD:SOT-23-3_GSD, symbol MOSFET_N_E
- removed Q2: MOSFET_N_E+P_E, M_SMD:SOT-23-6_G1-S2-G2-D2-S1-D1, symbol MOSFET_N_E+P_E
- removed U4: 74LVC1G07GW/V, M_SMD:SOT-23-5, symbol 74LVC1G07GW/V
- added Q1: MOSFET_N_E_Dual, M_SMD:SOT-23-6_G1-S2-G2-D2-S1-D1, symbol MOSFET_N_E_Dual
- added R10: 10, M_SMD:3225, symbol R
- R4: value 180 -> 1K
- R7: value 1K -> 5.6K
- R8, R9: value 10K -> 1K
- RN1, RN2, RN3: value 150 -> 270
- renumbered Q3 to Q2, Q4 to Q3, R10 to R11, R11 to R12, U5 to U4, U6 to U5
Connections:
- net SPEAKER is gone; now on net +5V: J1.20
- net +V_BATT: no longer R8.1
- net AUDIO_SIG: now also R9.2; no longer R9.1
- net GND: now also Q1.S1, Q1.S2; no longer J1.19, R9.2
- net MOTOR-: now also Q1.D1
- net MOTOR_SIG: now also R8.2
- new net: Q1.G1, R8.1
- new net: Q1.G2, R9.1
- new net: Q1.D2, R10.2
- new net SPEAKER-: J1.19, R10.1
Other:
- moved on the sheet: C13, C3, D1, R8, R9
